Commit message: Update code

File: src/quad_sim/urdf/quad_sim.xacro (robot description, xacro)
@@ -111,5 +111,5 @@
         <child link="propeller1" />
         <axis xyz="0 1 0" />
-        <dynamics damping="0.00" friction="0.00"/>
+        <dynamics damping="0.0004" friction="0.00"/>
     </joint>
     <propeller_link name="propeller2" />
@@ -119,5 +119,5 @@
         <child link="propeller2" />
         <axis xyz="0 1 0" />
-        <dynamics damping="0.00" friction="0.00"/>
+        <dynamics damping="0.0004" friction="0.00"/>
     </joint>
     <propeller_link name="propeller3" />
@@ -128,5 +128,5 @@
         <child link="propeller3" />
         <axis xyz="0 1 0" />
-        <dynamics damping="0.00" friction="0.00"/>
+        <dynamics damping="0.0004" friction="0.00"/>
     </joint>
     <propeller_link name="propeller4" />
@@ -136,5 +136,5 @@
         <child link="propeller4" />
         <axis xyz="0 1 0" />
-        <dynamics damping="0.00" friction="0.00"/>
+        <dynamics damping="0.0004" friction="0.00"/>
     </joint>
     <gazebo>

Commit message: Update Demo

File: src/quad_sim/urdf/quad_sim.xacro (robot description, xacro)
@@ -17,7 +17,7 @@
     </macro>
     <property name="PI" value="3.1415926535897931" />
-    <property name="frame_file_path" value="~/Quadrotor_Simulator/src/quad_sim/urdf/meshes/Frame_stl.stl" />
-    <property name="propeller_base_file_path" value="~/Quadrotor_Simulator/src/quad_sim/urdf/meshes/KV2540_Motor_Base.stl" />
-    <property name="propeller_file_path" value="~/Quadrotor_Simulator/src/quad_sim/urdf/meshes/KV2540_Motor_Propeller_holder.stl" />
+    <property name="frame_file_path" value="/home/nptttn/senior_project/quad_sim/src/quad_sim/urdf/meshes/final_frame.stl" />
+    <property name="propeller_base_file_path" value="/home/nptttn/senior_project/quad_sim/src/quad_sim/urdf/meshes/KV2540_Motor_Base.stl" />
+    <property name="propeller_file_path" value="/home/nptttn/senior_project/quad_sim/src/quad_sim/urdf/meshes/KV2540_Motor_Propeller_holder.stl" />
     <macro name="propeller_holder_link" params="name">
         <link name="${name}">
@@ -65,9 +65,9 @@
         <inertial>
             <mass value="0.061399" />
-            <origin xyz="0 0 0" rpy="0 0 0" />
+            <origin xyz="-0.11 0.11 0" rpy="0 0 0" />
             <frame_inertia />
         </inertial>
         <visual>
-            <origin xyz="0 0 0" rpy="0 0 0" />
+            <origin xyz="-0.11 0.11 0" rpy="${PI/2} 0 0" />
             <geometry>
                 <mesh filename="${frame_file_path}" scale="0.001 0.001 0.001" />
@@ -75,5 +75,5 @@
         </visual>
         <collision>
-            <origin xyz="0 0 0" rpy="0 0 0" />
+            <origin xyz="-0.11 0.11 0" rpy="${PI/2} 0 0" />
             <geometry>
                 <mesh filename="${frame_file_path}" scale="0.001 0.001 0.001" />
